Commit message: feat: extract arm model package structure

File: urdf/silverhand.urdf (robot description, URDF)
Before this commit: robot silverhand, 7 links, 6 joints
Joints:
- joint joint_2: origin xyz=0 0.064146 -0.16608 rpy=1.5708 0 -1.5708 -> xyz=0 0.064146 -0.16608 rpy=1.5708 0.5236 -1.5708
- joint joint_3: origin xyz=0.1525 -0.26414 0 rpy=0 0 0 -> xyz=0.1525 -0.26414 0 rpy=0 0 -1.0708

File: urdf/silverhand.urdf.xacro (robot description, xacro)
@@ -1,5 +1,6 @@
 <?xml version="1.0"?>
 <robot xmlns:xacro="http://www.ros.org/wiki/xacro" name="silverhand">
+  <xacro:arg name="arm_color" default="0.80 0.80 0.82 1"/>
   <xacro:include filename="$(find silverhand_arm_model)/urdf/silverhand_macro.urdf.xacro"/>
-  <xacro:silverhand_arm prefix=""/>
+  <xacro:silverhand_arm prefix="" color="$(arg arm_color)"/>
 </robot>

File: urdf/silverhand_macro.urdf.xacro (robot description, xacro)
@@ -1,5 +1,5 @@
 <?xml version="1.0"?>
 <robot name="silverhand_arm_macro" xmlns:xacro="http://www.ros.org/wiki/xacro">
-  <xacro:macro name="silverhand_arm" params="prefix parent:='' xyz:='0 0 0' rpy:='0 0 0'">
+  <xacro:macro name="silverhand_arm" params="prefix parent:='' xyz:='0 0 0' rpy:='0 0 0' color:='0.80 0.80 0.82 1'">
     <link name="${prefix}base_link">
       <inertial>
@@ -20,5 +20,5 @@
         </geometry>
         <material name="">
-          <color rgba="1 1 0 1"/>
+          <color rgba="${color}"/>
         </material>
       </visual>
@@ -55,5 +55,5 @@
         </geometry>
         <material name="">
-          <color rgba="1 1 0 1"/>
+          <color rgba="${color}"/>
         </material>
       </visual>
@@ -89,5 +89,5 @@
         </geometry>
         <material name="">
-          <color rgba="1 1 0 1"/>
+          <color rgba="${color}"/>
         </material>
       </visual>
@@ -123,5 +123,5 @@
         </geometry>
         <material name="">
-          <color rgba="1 1 0 1"/>
+          <color rgba="${color}"/>
         </material>
       </visual>
@@ -157,5 +157,5 @@
         </geometry>
         <material name="">
-          <color rgba="1 1 0 1"/>
+          <color rgba="${color}"/>
         </material>
       </visual>
@@ -191,5 +191,5 @@
         </geometry>
         <material name="">
-          <color rgba="1 1 0 1"/>
+          <color rgba="${color}"/>
         </material>
       </visual>
@@ -225,5 +225,5 @@
         </geometry>
         <material name="">
-          <color rgba="1 1 0 1"/>
+          <color rgba="${color}"/>
         </material>
       </visual>

Commit message: Adjust hardcoded zero pose for arm model

File: urdf/silverhand.urdf (robot description, URDF)
Before this commit: robot silverhand, 7 links, 6 joints
Joints:
- joint joint_2: origin xyz=0 0.064146 -0.16608 rpy=1.5708 0.5236 -1.5708 -> xyz=0 0.064146 -0.16608 rpy=1.5708 -1.0472 -1.5708
- joint joint_3: origin xyz=0.1525 -0.26414 0 rpy=0 0 -1.0708 -> xyz=0.1525 -0.26414 0 rpy=0 0 2.0708
- joint joint_5: origin xyz=0 0 -0.22225 rpy=3.1416 0 -2.8262 -> xyz=0 0 -0.22225 rpy=1.5708 0 -2.8262
- joint joint_6: origin xyz=-0.000294 0 0.02117 rpy=0 0 3.1416 -> xyz=-0.000294 0 0.02117 rpy=0 0 -1.5708

File: urdf/silverhand_macro.urdf.xacro (robot description, xacro)
@@ -100,5 +100,5 @@
     </link>
     <joint name="${prefix}joint_2" type="continuous">
-      <origin xyz="0 0.064146 -0.16608" rpy="1.5708 0.5236 -1.5708"/>
+      <origin xyz="0 0.064146 -0.16608" rpy="1.5708 -1.0472 -1.5708"/>
       <parent link="${prefix}link_1"/>
       <child link="${prefix}link_2"/>
@@ -134,5 +134,5 @@
     </link>
     <joint name="${prefix}joint_3" type="continuous">
-      <origin xyz="0.1525 -0.26414 0" rpy="0 0 -1.0708"/>
+      <origin xyz="0.1525 -0.26414 0" rpy="0 0 2.0708"/>
       <parent link="${prefix}link_2"/>
       <child link="${prefix}link_3"/>
@@ -202,5 +202,5 @@
     </link>
     <joint name="${prefix}joint_5" type="continuous">
-      <origin xyz="0 0 -0.22225" rpy="3.1416 0 -2.8262"/>
+      <origin xyz="0 0 -0.22225" rpy="1.5708 0 -2.8262"/>
       <parent link="${prefix}link_4"/>
       <child link="${prefix}link_5"/>
@@ -236,5 +236,5 @@
     </link>
     <joint name="${prefix}joint_6" type="continuous">
-      <origin xyz="-0.000294 0 0.02117" rpy="0 0 3.1416"/>
+      <origin xyz="-0.000294 0 0.02117" rpy="0 0 -1.5708"/>
       <parent link="${prefix}link_5"/>
       <child link="${prefix}link_6"/>
