Commit message: Refine arm base frame and rename URDF files

File: urdf/silverhand_macro.urdf.xacro (robot description, xacro)
@@ -2,5 +2,6 @@
 <robot name="silverhand_arm_macro" xmlns:xacro="http://www.ros.org/wiki/xacro">
   <xacro:macro name="silverhand_arm" params="prefix parent:='' xyz:='0 0 0' rpy:='0 0 0' color:='0.80 0.80 0.82 1'">
-    <link name="${prefix}base_link">
+    <link name="${prefix}base_link"/>
+    <link name="${prefix}arm_root_link">
       <inertial>
         <origin xyz="-4.6941E-06 0.054174 0.038824" rpy="0 0 0"/>
@@ -37,4 +38,9 @@
       </joint>
     </xacro:if>
+    <joint name="${prefix}arm_root_joint" type="fixed">
+      <origin xyz="0 0 0" rpy="0 0 1.5708"/>
+      <parent link="${prefix}base_link"/>
+      <child link="${prefix}arm_root_link"/>
+    </joint>
     <link name="${prefix}link_1">
       <inertial>
@@ -67,5 +73,5 @@
     <joint name="${prefix}joint_1" type="continuous">
       <origin xyz="0 0 0.003445" rpy="3.1416 0 0"/>
-      <parent link="${prefix}base_link"/>
+      <parent link="${prefix}arm_root_link"/>
       <child link="${prefix}link_1"/>
       <axis xyz="0 0 1"/>

Commit message: joints angle rotation adjusted

File: urdf/silverhand_macro.urdf.xacro (robot description, xacro)
@@ -75,5 +75,5 @@
       <parent link="${prefix}arm_root_link"/>
       <child link="${prefix}link_1"/>
-      <axis xyz="0 0 1"/>
+      <axis xyz="0 0 -1"/>
     </joint>
     <link name="${prefix}link_2">
@@ -211,5 +211,5 @@
       <parent link="${prefix}link_4"/>
       <child link="${prefix}link_5"/>
-      <axis xyz="-1 0 0"/>
+      <axis xyz="1 0 0"/>
     </joint>
     <link name="${prefix}link_6">

Commit message: Drop generated arm URDF from model package

File: urdf/silverhand_macro.urdf.xacro (robot description, xacro)
@@ -5,5 +5,5 @@
     <link name="${prefix}arm_root_link">
       <inertial>
-        <origin xyz="-4.6941E-06 0.054174 0.038824" rpy="0 0 0"/>
+        <origin xyz="0 0.054174 0.038824" rpy="0 0 0"/>
         <mass value="0.7102"/>
         <inertia
@@ -72,5 +72,5 @@
     </link>
     <joint name="${prefix}joint_1" type="continuous">
-      <origin xyz="0 0 0.003445" rpy="3.1416 0 0"/>
+      <origin xyz="0 0 0" rpy="3.1416 0 0"/>
       <parent link="${prefix}arm_root_link"/>
       <child link="${prefix}link_1"/>
@@ -113,5 +113,5 @@
     <link name="${prefix}link_3">
       <inertial>
-        <origin xyz="-0.00029765 -0.023661 -1.04720367321" rpy="0 0 0"/>
+        <origin xyz="0 -0.023661 -0.04720367321" rpy="0 0 0"/>
         <mass value="0.1787"/>
         <inertia
@@ -147,5 +147,5 @@
     <link name="${prefix}link_4">
       <inertial>
-        <origin xyz="-0.0016798 -0.00057319 -0.074404" rpy="0 0 0"/>
+        <origin xyz="0 0 -0.074404" rpy="0 0 0"/>
         <mass value="0.34936"/>
         <inertia
@@ -181,5 +181,5 @@
     <link name="${prefix}link_5">
       <inertial>
-        <origin xyz="0.0015066 -1.3102E-05 -0.012585" rpy="0 0 0"/>
+        <origin xyz="0.0015066 0 -0.012585" rpy="0 0 0"/>
         <mass value="0.11562"/>
         <inertia
@@ -215,5 +215,5 @@
     <link name="${prefix}link_6">
       <inertial>
-        <origin xyz="2.9287E-10 -1.6472E-09 0.0091432" rpy="0 0 0"/>
+        <origin xyz="0 0 0.01" rpy="0 0 0"/>
         <mass value="0.013863"/>
         <inertia
@@ -242,5 +242,5 @@
     </link>
     <joint name="${prefix}joint_6" type="continuous">
-      <origin xyz="-0.000294 0 0.02117" rpy="0 0 -1.5708"/>
+      <origin xyz="0 0 0.02117" rpy="0 0 -1.5708"/>
       <parent link="${prefix}link_5"/>
       <child link="${prefix}link_6"/>

Commit message: Support decoupled arm link and joint prefixes

File: urdf/silverhand_macro.urdf.xacro (robot description, xacro)
@@ -1,7 +1,15 @@
 <?xml version="1.0"?>
 <robot name="silverhand_arm_macro" xmlns:xacro="http://www.ros.org/wiki/xacro">
-  <xacro:macro name="silverhand_arm" params="prefix parent:='' xyz:='0 0 0' rpy:='0 0 0' color:='0.80 0.80 0.82 1'">
-    <link name="${prefix}base_link"/>
-    <link name="${prefix}arm_root_link">
+  <xacro:macro
+    name="silverhand_arm"
+    params="prefix:='' joint_prefix:='__default__' link_prefix:='__default__' parent:='' xyz:='0 0 0' rpy:='0 0 0' color:='0.80 0.80 0.82 1'">
+    <xacro:property
+      name="resolved_joint_prefix"
+      value="${prefix if joint_prefix == '__default__' else joint_prefix}"/>
+    <xacro:property
+      name="resolved_link_prefix"
+      value="${prefix if link_prefix == '__default__' else link_prefix}"/>
+    <link name="${resolved_link_prefix}base_link"/>
+    <link name="${resolved_link_prefix}arm_root_link">
       <inertial>
         <origin xyz="0 0.054174 0.038824" rpy="0 0 0"/>
@@ -32,16 +40,16 @@
     </link>
     <xacro:if value="${parent != ''}">
-      <joint name="${prefix}mount_joint" type="fixed">
+      <joint name="${resolved_joint_prefix}mount_joint" type="fixed">
         <origin xyz="${xyz}" rpy="${rpy}"/>
         <parent link="${parent}"/>
-        <child link="${prefix}base_link"/>
+        <child link="${resolved_link_prefix}base_link"/>
       </joint>
     </xacro:if>
-    <joint name="${prefix}arm_root_joint" type="fixed">
+    <joint name="${resolved_joint_prefix}arm_root_joint" type="fixed">
       <origin xyz="0 0 0" rpy="0 0 1.5708"/>
-      <parent link="${prefix}base_link"/>
-      <child link="${prefix}arm_root_link"/>
-    </joint>
-    <link name="${prefix}link_1">
+      <parent link="${resolved_link_prefix}base_link"/>
+      <child link="${resolved_link_prefix}arm_root_link"/>
+    </joint>
+    <link name="${resolved_link_prefix}link_1">
       <inertial>
         <origin xyz="-0.022706 0.04294 -0.12205" rpy="0 0 0"/>
@@ -71,11 +79,11 @@
       </collision>
     </link>
-    <joint name="${prefix}joint_1" type="continuous">
+    <joint name="${resolved_joint_prefix}joint_1" type="continuous">
       <origin xyz="0 0 0" rpy="3.1416 0 0"/>
-      <parent link="${prefix}arm_root_link"/>
-      <child link="${prefix}link_1"/>
-      <axis xyz="0 0 -1"/>
-    </joint>
-    <link name="${prefix}link_2">
+      <parent link="${resolved_link_prefix}arm_root_link"/>
+      <child link="${resolved_link_prefix}link_1"/>
+      <axis xyz="0 0 -1"/>
+    </joint>
+    <link name="${resolved_link_prefix}link_2">
       <inertial>
         <origin xyz="0.064818 -0.11189 -0.038671" rpy="0 0 0"/>
@@ -105,11 +113,11 @@
       </collision>
     </link>
-    <joint name="${prefix}joint_2" type="continuous">
+    <joint name="${resolved_joint_prefix}joint_2" type="continuous">
       <origin xyz="0 0.064146 -0.16608" rpy="1.5708 -1.0472 -1.5708"/>
-      <parent link="${prefix}link_1"/>
-      <child link="${prefix}link_2"/>
-      <axis xyz="0 0 -1"/>
-    </joint>
-    <link name="${prefix}link_3">
+      <parent link="${resolved_link_prefix}link_1"/>
+      <child link="${resolved_link_prefix}link_2"/>
+      <axis xyz="0 0 -1"/>
+    </joint>
+    <link name="${resolved_link_prefix}link_3">
       <inertial>
         <origin xyz="0 -0.023661 -0.04720367321" rpy="0 0 0"/>
@@ -139,11 +147,11 @@
       </collision>
     </link>
-    <joint name="${prefix}joint_3" type="continuous">
+    <joint name="${resolved_joint_prefix}joint_3" type="continuous">
       <origin xyz="0.1525 -0.26414 0" rpy="0 0 2.0708"/>
-      <parent link="${prefix}link_2"/>
-      <child link="${prefix}link_3"/>
-      <axis xyz="0 0 -1"/>
-    </joint>
-    <link name="${prefix}link_4">
+      <parent link="${resolved_link_prefix}link_2"/>
+      <child link="${resolved_link_prefix}link_3"/>
+      <axis xyz="0 0 -1"/>
+    </joint>
+    <link name="${resolved_link_prefix}link_4">
       <inertial>
         <origin xyz="0 0 -0.074404" rpy="0 0 0"/>
@@ -173,11 +181,11 @@
       </collision>
     </link>
-    <joint name="${prefix}joint_4" type="continuous">
+    <joint name="${resolved_joint_prefix}joint_4" type="continuous">
       <origin xyz="0 0 0.00675" rpy="1.5708 -1.2554 -1.5708"/>
-      <parent link="${prefix}link_3"/>
-      <child link="${prefix}link_4"/>
-      <axis xyz="0 0 -1"/>
-    </joint>
-    <link name="${prefix}link_5">
+      <parent link="${resolved_link_prefix}link_3"/>
+      <child link="${resolved_link_prefix}link_4"/>
+      <axis xyz="0 0 -1"/>
+    </joint>
+    <link name="${resolved_link_prefix}link_5">
       <inertial>
         <origin xyz="0.0015066 0 -0.012585" rpy="0 0 0"/>
@@ -207,11 +215,11 @@
       </collision>
     </link>
-    <joint name="${prefix}joint_5" type="continuous">
+    <joint name="${resolved_joint_prefix}joint_5" type="continuous">
       <origin xyz="0 0 -0.22225" rpy="1.5708 0 -2.8262"/>
-      <parent link="${prefix}link_4"/>
-      <child link="${prefix}link_5"/>
+      <parent link="${resolved_link_prefix}link_4"/>
+      <child link="${resolved_link_prefix}link_5"/>
       <axis xyz="1 0 0"/>
     </joint>
-    <link name="${prefix}link_6">
+    <link name="${resolved_link_prefix}link_6">
       <inertial>
         <origin xyz="0 0 0.01" rpy="0 0 0"/>
@@ -241,8 +249,8 @@
       </collision>
     </link>
-    <joint name="${prefix}joint_6" type="continuous">
+    <joint name="${resolved_joint_prefix}joint_6" type="continuous">
       <origin xyz="0 0 0.02117" rpy="0 0 -1.5708"/>
-      <parent link="${prefix}link_5"/>
-      <child link="${prefix}link_6"/>
+      <parent link="${resolved_link_prefix}link_5"/>
+      <child link="${resolved_link_prefix}link_6"/>
       <axis xyz="0 0 1"/>
     </joint>
